Commit message: ...

File: src/maze_bot_description/urdf/maze_bot.urdf.xacro (robot description, xacro)
@@ -1,8 +1,8 @@
 <?xml version="1.0"?>
 <robot xmlns:xacro="http://www.ros.org/wiki/xacro" name="maze_bot">
-  <!-- Define robot parameters -->
-  <xacro:property name="base_width" value="0.31"/>
-  <xacro:property name="base_length" value="0.42"/>
-  <xacro:property name="base_height" value="0.18"/>
+  <!-- Define robot parameters - Optimized for stability -->
+  <xacro:property name="base_width" value="0.40"/>   <!-- Increased for stability -->
+  <xacro:property name="base_length" value="0.45"/>  <!-- Slightly increased -->
+  <xacro:property name="base_height" value="0.12"/>  <!-- Lowered center of mass -->
   <xacro:property name="wheel_radius" value="0.10"/>
   <xacro:property name="wheel_width" value="0.04"/>
@@ -47,5 +47,5 @@
       </geometry>
     </collision>
-    <xacro:box_inertia m="15" w="${base_width}" d="${base_length}" h="${base_height}"/>
+    <xacro:box_inertia m="8.0" w="${base_width}" d="${base_length}" h="${base_height}"/>
   </link>
   <!-- Robot Footprint -->
@@ -74,5 +74,5 @@
         </geometry>
       </collision>
-      <xacro:cylinder_inertia m="0.5" r="${wheel_radius}" h="${wheel_width}"/>
+      <xacro:cylinder_inertia m="1.2" r="${wheel_radius}" h="${wheel_width}"/>
     </link>
     <joint name="${prefix}_joint" type="continuous">
@@ -101,5 +101,5 @@
       </geometry>
     </collision>
-    <xacro:sphere_inertia m="0.5" r="${(wheel_radius+wheel_zoff-(base_height/2))}"/>
+    <xacro:sphere_inertia m="0.8" r="${(wheel_radius+wheel_zoff-(base_height/2))}"/>
   </link>
   <joint name="caster_joint" type="fixed">

File: src/maze_bot_description/urdf/maze_bot_gazebo.xacro (robot description, xacro)
@@ -65,10 +65,28 @@
   <gazebo reference="base_link">
     <material>Gazebo/Blue</material>
+    <mu1>0.8</mu1>
+    <mu2>0.8</mu2>
+    <kp>1000000.0</kp>
+    <kd>100.0</kd>
+    <minDepth>0.001</minDepth>
+    <maxVel>1.0</maxVel>
   </gazebo>
   <gazebo reference="drivewhl_l_link">
     <material>Gazebo/Black</material>
+    <mu1>1.5</mu1>
+    <mu2>1.5</mu2>
+    <kp>1000000.0</kp>
+    <kd>100.0</kd>
+    <minDepth>0.001</minDepth>
+    <maxVel>1.0</maxVel>
   </gazebo>
   <gazebo reference="drivewhl_r_link">
     <material>Gazebo/Black</material>
+    <mu1>1.5</mu1>
+    <mu2>1.5</mu2>
+    <kp>1000000.0</kp>
+    <kd>100.0</kd>
+    <minDepth>0.001</minDepth>
+    <maxVel>1.0</maxVel>
   </gazebo>
   <gazebo reference="front_caster">
